File: Yet Another Modified Redox.kicad_pcb (KiCad board)
At the start: 2 copper layers, 370.6 x 126 mm, 179 parts, among them J1 USB_B_Mini, J2 AudioJack4, J3 AudioJack4, K1 KEYSW, K10 KEYSW, K11 KEYSW, K12 KEYSW, K13 KEYSW, K14 KEYSW, K15 KEYSW, K16 KEYSW, K17 KEYSW, K18 KEYSW, K19 KEYSW, K2 KEYSW, K20 KEYSW, K21 KEYSW, K22 KEYSW, K23 KEYSW, K24 KEYSW, K25 KEYSW, K26 KEYSW, K27 KEYSW, K28 KEYSW, K29 KEYSW, K3 KEYSW, K30 KEYSW, K31 KEYSW, K32 KEYSW, K33 KEYSW, K34 KEYSW, K35 KEYSW, K36 KEYSW, K37 KEYSW, K38 KEYSW, K39 KEYSW, K4 KEYSW, K40 KEYSW, K41 KEYSW, K42 KEYSW, K43 KEYSW, K44 KEYSW, K45 KEYSW, K46 KEYSW, K47 KEYSW, K48 KEYSW, K49 KEYSW, K5 KEYSW, K50 KEYSW, K51 KEYSW, K52 KEYSW, K53 KEYSW, K54 KEYSW, K55 KEYSW, K56 KEYSW, K57 KEYSW, K58 KEYSW, K59 KEYSW, K6 KEYSW, K60 KEYSW, K61 KEYSW, K62 KEYSW, K63 KEYSW, K64 KEYSW, K65 KEYSW, K66 KEYSW, K67 KEYSW, K68 KEYSW, K69 KEYSW, K7 KEYSW, K70 KEYSW, K8 KEYSW, K9 KEYSW, Q1 DMG2302U, Q2 DMG2302U, Q3 DMG2302U, U1 YAAJ_BluePill_Part_Like, U2 YAAJ_BluePill_Part_Like

Commit message: Update to use rp2040 stamp
Parts:
- removed D74, D75: D_Schottky, Diode_SMD:D_SOD-123
- removed the REF** at (33.3, 33.3)
- removed the REF** at (133.3, 33.3)
- removed the REF** at (33.3, 128.6)
- removed the REF** at (204.8, 123.8)
- added C4: 1uF, Capacitor_SMD:C_0805_2012Metric, F.Cu at (234.6, 63.2)
- added C5: 1uF, Capacitor_SMD:C_0805_2012Metric, F.Cu at (193.9, 41.5)
- added H6: MountingHole_3.2mm_M3_ISO14580_Pad, MountingHole:MountingHole_3.2mm_M3_ISO14580_Pad, F.Cu at (133.3, 33.3)
- added H7: MountingHole_3.2mm_M3_ISO14580_Pad, MountingHole:MountingHole_3.2mm_M3_ISO14580_Pad, F.Cu at (33.3, 33.3)
- added H8: MountingHole_3.2mm_M3_ISO14580_Pad, MountingHole:MountingHole_3.2mm_M3_ISO14580_Pad, F.Cu at (33.3, 128.6)
- added H9: MountingHole_3.2mm_M3_ISO14580_Pad, MountingHole:MountingHole_3.2mm_M3_ISO14580_Pad, F.Cu at (204.8, 123.8)
- added R10: 10kR, Resistor_SMD:R_0805_2012Metric, F.Cu at (198.1, 42.1)
- added R11: 10kR, Resistor_SMD:R_0805_2012Metric, F.Cu at (198.1, 40.0)
- added R12: 1kR, Resistor_SMD:R_0805_2012Metric, F.Cu at (224.8, 80.7)
- added R13: 1kR, Resistor_SMD:R_0805_2012Metric, F.Cu at (224.8, 78.7)
- added R14: 20R, Resistor_SMD:R_0805_2012Metric, F.Cu at (185.9, 41.7)
- added R15: 20R, Resistor_SMD:R_0805_2012Metric, F.Cu at (187.9, 41.7)
- added R16: 100R, Resistor_SMD:R_0805_2012Metric, F.Cu at (229.0, 84.3)
- added SW1: SW_Push, Button_Switch_SMD:SW_SPST_SKQG_WithoutStem, F.Cu at (205.2, 62.4)
- added TP1: TP, TestPoint:TestPoint_Pad_D2.0mm, F.Cu at (182.0, 38.4)
- added TP2: TestPoint, TestPoint:TestPoint_Pad_D2.0mm, F.Cu at (178.2, 38.5)
- U1: value YAAJ_BluePill_Part_Like -> CY8C9540A-IOExpander; footprint Footprints:YAAJ_BluePill_1 -> Package_SO:SSOP-48_7.5x15.9mm_P0.635mm
- U2: value YAAJ_BluePill_Part_Like -> RP2040_Stamp; footprint Footprints:YAAJ_BluePill_1 -> RP2040_Stamp:RP2040_Stamp_SMD
- moved U1 62.7 mm to (234.7, 75.1)
- moved U2 48.6 mm to (186.9, 57.2)
- renumbered REF** to H10, REF** to H2, REF** to H3, REF** to H4, REF** to H5
Connections:
- net Net-(C1-Pad1) renamed /VBUS
- J1 pad 4: (no net) -> unconnected-(J1-Pad4)
- J2 pad R1: /TX -> /SCL_M
- J2 pad R2: (no net) -> /SDA_M
- J3 pad R1: /RX -> /SCL_S
- J3 pad R2: (no net) -> /SDA_S
- U1 pad 1: /NUM_LOCK -> /RR1
- U1 pad 10: (no net) -> unconnected-(U1-Pad10)
- U1 pad 11: /LC1 -> unconnected-(U1-Pad11)
- U1 pad 12: /LC2 -> unconnected-(U1-Pad12)
- U1 pad 13: /LC3 -> /RGND
- U1 pad 14: /LC4 -> unconnected-(U1-Pad14)
- U1 pad 15: /LC5 -> unconnected-(U1-Pad15)
- U1 pad 16: /LC6 -> unconnected-(U1-Pad16)
- U1 pad 17: /LC7 -> unconnected-(U1-Pad17)
- U1 pad 18: /L+5V -> unconnected-(U1-Pad18)
- U1 pad 19: /LGND -> unconnected-(U1-Pad19)
- U1 pad 2: /CAPSLOCK -> /RR2
- U1 pad 20: (no net) -> /SCL_S
- U1 pad 21: (no net) -> /SDA_S
- U1 pad 22: (no net) -> unconnected-(U1-Pad22)
- U1 pad 23: (no net) -> Net-(R16-Pad1)
- U1 pad 24: (no net) -> /RGND
- U1 pad 25: /LR1 -> unconnected-(U1-Pad25)
- U1 pad 26: /LR2 -> unconnected-(U1-Pad26)
- U1 pad 27: /LR3 -> unconnected-(U1-Pad27)
- U1 pad 28: /LR4 -> unconnected-(U1-Pad28)
- U1 pad 29: /LR5 -> unconnected-(U1-Pad29)
- U1 pad 3: /SCROLL_LOCK -> /RR3
- U1 pad 30: (no net) -> unconnected-(U1-Pad30)
- U1 pad 31: (no net) -> unconnected-(U1-Pad31)
- U1 pad 32: (no net) -> unconnected-(U1-Pad32)
- U1 pad 33: (no net) -> unconnected-(U1-Pad33)
- U1 pad 34: (no net) -> unconnected-(U1-Pad34)
- U1 pad 35: (no net) -> unconnected-(U1-Pad35)
- U1 pad 36: (no net) -> unconnected-(U1-Pad36)
- U1 pad 37: (no net) -> unconnected-(U1-Pad37)
- U1 pad 38: (no net) -> unconnected-(U1-Pad38)
- U1 pad 39: /LGND -> unconnected-(U1-Pad39)
- U1 pad 4: /TX -> /RR4
- U1 pad 40: /LGND -> unconnected-(U1-Pad40)
- U1 pad 5: (no net) -> /RR5
- U1 pad 6: (no net) -> unconnected-(U1-Pad6)
- U1 pad 7: (no net) -> unconnected-(U1-Pad7)
- U1 pad 8: /D- -> unconnected-(U1-Pad8)
- U1 pad 9: /D+ -> unconnected-(U1-Pad9)
- U2 pad 1: (no net) -> /SDA_M
- U2 pad 10: (no net) -> /LC3
- U2 pad 11: /RC1 -> /LC4
- U2 pad 12: /RC2 -> /LC5
- U2 pad 13: /RC3 -> /LC6
- U2 pad 14: /RC4 -> /LC7
- U2 pad 15: /RC5 -> /NUM_LOCK
- U2 pad 16: /RC6 -> /CAPSLOCK
- U2 pad 17: /RC7 -> /SCROLL_LOCK
- U2 pad 18: /R+5V -> unconnected-(U2-Pad18)
- U2 pad 19: /RGND -> unconnected-(U2-Pad19)
- U2 pad 2: (no net) -> /SCL_M
- U2 pad 20: (no net) -> unconnected-(U2-Pad20)
- U2 pad 21: (no net) -> unconnected-(U2-Pad21)
- U2 pad 22: (no net) -> unconnected-(U2-Pad22)
- U2 pad 23: (no net) -> unconnected-(U2-Pad23)
- U2 pad 24: (no net) -> unconnected-(U2-Pad24)
- U2 pad 25: /RR1 -> unconnected-(U2-Pad25)
- U2 pad 26: /RR2 -> unconnected-(U2-Pad26)
- U2 pad 27: /RR3 -> unconnected-(U2-Pad27)
- U2 pad 28: /RR4 -> unconnected-(U2-Pad28)
- U2 pad 29: /RR5 -> unconnected-(U2-Pad29)
- U2 pad 3: (no net) -> /LR1
- U2 pad 30: (no net) -> unconnected-(U2-Pad30)
- U2 pad 31: (no net) -> /LGND
- U2 pad 32: (no net) -> unconnected-(U2-Pad32)
- U2 pad 33: (no net) -> /L+5V
- U2 pad 34: (no net) -> unconnected-(U2-Pad34)
- U2 pad 35: (no net) -> /D_C-
- U2 pad 36: (no net) -> /D_C+
- U2 pad 37: (no net) -> Net-(TP1-Pad1)
- U2 pad 38: (no net) -> Net-(TP2-Pad1)
- U2 pad 39: /RGND -> unconnected-(U2-Pad39)
- U2 pad 4: /RX -> /LR2
- U2 pad 40: /RGND -> Net-(SW1-Pad2)
- U2 pad 5: (no net) -> /LR3
- U2 pad 6: (no net) -> /LR4
- U2 pad 7: (no net) -> /LR5
- U2 pad 8: (no net) -> /LC1
- U2 pad 9: (no net) -> /LC2
Routing:
- net /SDA_S: track 0.00 -> 61.8 mm, vias 0 -> 1
- net /SCL_S: track 0.00 -> 53.8 mm, vias 0 -> 1
- net /SDA_M: track 0.00 -> 49.1 mm, vias 0 -> 2
- net /LR1: track 205.0 -> 156.5 mm, vias 2 -> 0
- net /SCL_M: track 0.00 -> 44.3 mm, vias 0 -> 2
- net /L+5V: track 116.7 -> 74.6 mm
- net Net-(SW1-Pad2): track 0.00 -> 38.6 mm, vias 0 -> 2
- net /TX: track 32.6 -> 0.00 mm
- net /SCROLL_LOCK: track 36.8 -> 65.1 mm, vias 0 -> 1
- net /CAPSLOCK: track 27.5 -> 54.7 mm, vias 0 -> 1
- net /NUM_LOCK: track 17.0 -> 43.0 mm, vias 0 -> 1
- net /D+: track 37.2 -> 13.2 mm, vias 3 -> 2
- net /RR3: track 167.5 -> 191.1 mm
- net /D-: track 35.1 -> 12.9 mm, vias 4 -> 2
- net /RX: track 21.7 -> 0.00 mm
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Other:
- board size 370.6 x 126 mm -> 370.6 x 125.8 mm
- net class Default removed
- board text added: "v0.1.0 12/26/21"
- board text removed: "v0.0.1 03/15/21"
