File: Yet Another Modified Redox.sch (KiCad schematic (older format))
At the start: 167 parts, among them J1 USB_B_Mini, J2 AudioJack4, J3 AudioJack4, K1 KEYSW, K10 KEYSW, K11 KEYSW, K12 KEYSW, K13 KEYSW, K14 KEYSW, K15 KEYSW, K16 KEYSW, K17 KEYSW, K18 KEYSW, K19 KEYSW, K2 KEYSW, K20 KEYSW, K21 KEYSW, K22 KEYSW, K23 KEYSW, K24 KEYSW, K25 KEYSW, K26 KEYSW, K27 KEYSW, K28 KEYSW, K29 KEYSW, K3 KEYSW, K30 KEYSW, K31 KEYSW, K32 KEYSW, K33 KEYSW, K34 KEYSW, K35 KEYSW, K36 KEYSW, K37 KEYSW, K38 KEYSW, K39 KEYSW, K4 KEYSW, K40 KEYSW, K41 KEYSW, K42 KEYSW, K43 KEYSW, K44 KEYSW, K45 KEYSW, K46 KEYSW, K47 KEYSW, K48 KEYSW, K49 KEYSW, K5 KEYSW, K50 KEYSW, K51 KEYSW, K52 KEYSW, K53 KEYSW, K54 KEYSW, K55 KEYSW, K56 KEYSW, K57 KEYSW, K58 KEYSW, K59 KEYSW, K6 KEYSW, K60 KEYSW, K61 KEYSW, K62 KEYSW, K63 KEYSW, K64 KEYSW, K65 KEYSW, K66 KEYSW, K67 KEYSW, K68 KEYSW, K69 KEYSW, K7 KEYSW, K70 KEYSW, K8 KEYSW, K9 KEYSW, Q1 DMG2302U, Q2 DMG2302U, Q3 DMG2302U, U1 YAAJ_BluePill_Part_Like, U2 YAAJ_BluePill_Part_Like

Commit message: Update to use rp2040 stamp
Parts:
- removed D74, D75: D_Schottky, Diode_SMD:D_SOD-123, symbol Device:D_Schottky
- removed U1, U2: YAAJ_BluePill_Part_Like, Footprints:YAAJ_BluePill_1, symbol YAAJ_BluePill_Part_Like:YAAJ_BluePill_Part_Like
- added C4, C5: 1uF, Capacitor_SMD:C_0805_2012Metric, symbol Device:C
- added H1, H10, H2, H3, H4, H5, H6, H7, H8, H9: M3, MountingHole:MountingHole_3.2mm_M3_ISO14580_Pad, symbol Mechanical:MountingHole_Pad
- added R10, R11: 10kR, Resistor_SMD:R_0805_2012Metric, symbol Device:R
- added R12, R13: 1kR, Resistor_SMD:R_0805_2012Metric, symbol Device:R
- added R14, R15: 20R, Resistor_SMD:R_0805_2012Metric, symbol Device:R
- added R16: 100R, Resistor_SMD:R_0805_2012Metric, symbol Device:R
- added SW1: SW_Push, Button_Switch_SMD:SW_SPST_SKQG_WithoutStem, symbol Switch:SW_Push
- added TP1: TP, TestPoint:TestPoint_Pad_D2.0mm, symbol Connector:TestPoint
- added TP2: TestPoint, TestPoint:TestPoint_Pad_D2.0mm, symbol Connector:TestPoint
- added U1: CY8C9540A-IOExpander, Package_SO:SSOP-48_7.5x15.9mm_P0.635mm, symbol WM_lib:CY8C9540A-IOExpander
- added U2: RP2040_Stamp, RP2040_Stamp:RP2040_Stamp_SMD, symbol RP2040_Stamp:RP2040_Stamp
- J1: symbol Connector:USB_B_Mini -> Yet-Another-Modified-Redox-rescue:USB_B_Mini-Connector
- K1, K10, K11, K12, K13, K14, K15, K16, K17, K18, K19, K2, K20, K21, K22, K23, K24, K25, K26, K27, K28, K29, K3, K30, K31, K32, K33, K34, K35, K36, K37, K38, K39, K4, K40, K41, K42, K43, K44, K45, K46, K47, K48, K49, K5, K50, K51, K52, K53, K54, K55, K56, K57, K58, K59, K6, K60, K61, K62, K63, K64, K65, K66, K67, K68, K69, K7, K70, K8, K9: symbol keyboard_parts:KEYSW -> Yet-Another-Modified-Redox-rescue:KEYSW-keyboard_parts
Connections:
- net CAPSLOCK: now also U2.16 (GPIO15)
- net D+: now also R14.2
- net D-: now also R15.1
- net L+5V: now also C5.1, R10.2, R11.1, U2.33 (5V)
- net LC1: now also U2.8 (GPIO7)
- net LC2: now also U2.9 (GPIO8)
- net LC3: now also U2.10 (GPIO9)
- net LC4: now also U2.11 (GPIO10)
- net LC5: now also U2.12 (GPIO11)
- net LC6: now also U2.13 (GPIO12)
- net LC7: now also U2.14 (GPIO13)
- net LGND: now also C5.2, H10.1, H6.1, H7.1, H8.1, H9.1, SW1.1, U2.31 (GND)
- net LR1: now also U2.3 (GPIO2)
- net LR2: now also U2.4 (GPIO3)
- net LR3: now also U2.5 (GPIO4)
- net LR4: now also U2.6 (GPIO5)
- net LR5: now also U2.7 (GPIO6)
- net NUM_LOCK: now also U2.15 (GPIO14)
- net R+5V: now also C4.1, R12.2, R13.1, U1.48 (VDD)
- net RC1: now also U1.47 (GP1_0_PWM6)
- net RC2: now also U1.46 (GP1_1_PWM4)
- net RC3: now also U1.45 (GP1_2_PWM2)
- net RC4: now also U1.44 (GP1_3_PWM0)
- net RC5: now also U1.43 (GP1_4_PWM6)
- net RC6: now also U1.42 (GP1_5_PWM4/A6)
- net RC7: now also U1.41 (GP1_6_PWM2/A5)
- net RGND: now also C4.2, H1.1, H2.1, H3.1, H4.1, H5.1, R16.2, U1.13 (VSS), U1.24 (VSS)
- net RR1: now also U1.1 (GP0_0_PWM7)
- net RR2: now also U1.2 (GP0_1_PWM5)
- net RR3: now also U1.3 (GP0_2_PWM3)
- net RR4: now also U1.4 (GP0_3_PWM1)
- net RR5: now also U1.5 (GP0_4_PWM7)
- net SCROLL_LOCK: now also U2.17 (GPIO16)
- net SDA_M: now reaches J2.R2
- net SDA_M: now also R10.1, U2.1 (GPIO0)
- net SDA_S: now reaches J3.R2
- net SDA_S: now also R12.1, U1.21 (SDA)
- net VBUS: now reaches C1.1, J1.1 (VBUS), L1.1
- net RX renamed SCL_S
- net SCL_S: now also R13.2, U1.20 (SCL)
- net TX renamed SCL_M
- net SCL_M: now also R11.2, U2.2 (GPIO1)
- new net: TP1.1, U2.37 (SWDIO)
- new net: TP2.1, U2.38 (SWCLK)
- new net: SW1.2, U2.40 (BOOTSEL)
- new net: R16.1, U1.23 (A0)
- new net D_C+: R14.1, U2.35 (USB_D-)
- new net D_C-: R15.2, U2.36 (USB_D+)
- no-connect marks 44 -> 47
Other:
- note added: "Left Control"
- note added: "Right Control"
- note removed: "Left Controller"
- note removed: "Right Controller"
- moved on the sheet: C1, C2, C3, D76, J1, J2, J3, L1
